File: KiCAD/CIB - Sandbird Octopus.kicad_pcb (KiCad board)
At the start: 2 copper layers, 73 x 55.9 mm, 51 parts, among them J1 DA15, J2 Molex, J3 PT 3-4, J4 PT 1-2, J5 Enable, J6 Pin Header, Q1 STN3NF06, Q2 STN3NF06, Q3 STN3NF06, Q4 STN3NF06, Q5 STN3NF06

Commit message: .
Parts:
- moved J4 31.0 mm to (144.1, 86.4)
- moved K5 7.62 mm to (119.5, 50.8)

Commit message: .
Parts:
- removed J2: Molex, Connector_Molex:Molex_Micro-Fit_3.0_43045-1018_2x05-1MP_P3.00mm_Vertical
- removed J3: PT 3-4, TerminalBlock_Phoenix:TerminalBlock_Phoenix_MPT-0,5-4-2.54_1x04_P2.54mm_Horizontal
- removed J4: PT 1-2, TerminalBlock_Phoenix:TerminalBlock_Phoenix_MPT-0,5-4-2.54_1x04_P2.54mm_Horizontal
- added D14: Red, LED_SMD:LED_0805_2012Metric_Pad1.15x1.40mm_HandSolder, F.Cu at (84.5, 49.9)
- added D15: Red, LED_SMD:LED_0805_2012Metric_Pad1.15x1.40mm_HandSolder, F.Cu at (84.5, 53.0)
- added D16: Red, LED_SMD:LED_0805_2012Metric_Pad1.15x1.40mm_HandSolder, F.Cu at (84.5, 56.0)
- added Q6: STN3NF06, Package_TO_SOT_SMD:SOT-223-3_TabPin2, F.Cu at (77.1, 52.6)
- added Q7: STN3NF06, Package_TO_SOT_SMD:SOT-223-3_TabPin2, F.Cu at (77.1, 60.9)
- added Q8: STN3NF06, Package_TO_SOT_SMD:SOT-223-3_TabPin2, F.Cu at (77.1, 69.2)
- added R19: 1k, Resistor_SMD:R_0805_2012Metric_Pad1.20x1.40mm_HandSolder, F.Cu at (69.8, 49.9)
- added R20: 10k, Resistor_SMD:R_0805_2012Metric_Pad1.20x1.40mm_HandSolder, F.Cu at (69.8, 52.8)
- added R21: 1k, Resistor_SMD:R_0805_2012Metric_Pad1.20x1.40mm_HandSolder, F.Cu at (69.8, 55.8)
- added R22: 1k, Resistor_SMD:R_0805_2012Metric_Pad1.20x1.40mm_HandSolder, F.Cu at (69.8, 58.7)
- added R23: 10k, Resistor_SMD:R_0805_2012Metric_Pad1.20x1.40mm_HandSolder, F.Cu at (69.8, 61.7)
- added R24: 1k, Resistor_SMD:R_0805_2012Metric_Pad1.20x1.40mm_HandSolder, F.Cu at (69.8, 64.6)
- added R25: 1k, Resistor_SMD:R_0805_2012Metric_Pad1.20x1.40mm_HandSolder, F.Cu at (69.8, 67.6)
- added R26: 10k, Resistor_SMD:R_0805_2012Metric_Pad1.20x1.40mm_HandSolder, F.Cu at (69.8, 70.5)
- added R27: 1k, Resistor_SMD:R_0805_2012Metric_Pad1.20x1.40mm_HandSolder, F.Cu at (69.8, 73.5)
- J1: value DA15 -> DB25; footprint Connector_Dsub:DSUB-9_Female_Horizontal_P2.77x2.84mm_EdgePinOffset7.70mm_Housed_MountingHolesOffset9.12mm -> Connector_Dsub:DSUB-25_Socket_Horizontal_P2.77x2.84mm_EdgePinOffset7.70mm_Housed_MountingHolesOffset9.12mm
- J6: value Pin Header -> Conn_01x26_Pin
- moved J1 10.3 mm to (152.4, 48.1)
Connections:
- J1 pad 1: /PT1 in -> /Pin_01
- J1 pad 2: /PT2 in -> /Pin_02
- J1 pad 3: /PT3 in -> /Pin_03
- J1 pad 4: /PT4 in -> /Pin_04
- J1 pad 6: /PT1 out -> /Pin_06
- J1 pad 7: /PT2 out -> /Pin_07
- J1 pad 8: /PT3 out -> /Pin_08
- J1 pad 9: /PT4 out -> /Pin_09
- J6 pad 1: /PT1 in -> /Pin_01
- J6 pad 10: GND -> /Pin_18
- J6 pad 2: /PT1 out -> /Pin_14
- J6 pad 3: /PT2 in -> /Pin_02
- J6 pad 4: /PT2 out -> /Pin_15
- J6 pad 5: /PT3 in -> /Pin_03
- J6 pad 6: /PT3 out -> /Pin_16
- J6 pad 7: /PT4 in -> /Pin_04
- J6 pad 8: /PT4 out -> /Pin_17
- K1 pad 2: unconnected-(K1-Pad2) -> /Pin_16
- K1 pad 3: unconnected-(K1-Pad3) -> /Pin_03
- K1 pad 4: unconnected-(K1-Pad4) -> /Pin_15
- K1 pad 5: unconnected-(K1-Pad5) -> /Pin_01
- K1 pad 6: unconnected-(K1-Pad6) -> /Pin_14
- K1 pad 7: unconnected-(K1-Pad7) -> /Pin_02
- K2 pad 2: unconnected-(K2-Pad2) -> /Pin_19
- K2 pad 3: unconnected-(K2-Pad3) -> /Pin_06
- K2 pad 4: unconnected-(K2-Pad4) -> /Pin_18
- K2 pad 5: unconnected-(K2-Pad5) -> /Pin_04
- K2 pad 6: unconnected-(K2-Pad6) -> /Pin_17
- K2 pad 7: unconnected-(K2-Pad7) -> /Pin_05
- K3 pad 2: unconnected-(K3-Pad2) -> /Pin_22
- K3 pad 3: unconnected-(K3-Pad3) -> /Pin_09
- K3 pad 4: unconnected-(K3-Pad4) -> /Pin_21
- K3 pad 5: unconnected-(K3-Pad5) -> /Pin_07
- K3 pad 6: unconnected-(K3-Pad6) -> /Pin_20
- K3 pad 7: unconnected-(K3-Pad7) -> /Pin_08
- K4 pad 2: unconnected-(K4-Pad2) -> /Pin_25
- K4 pad 3: unconnected-(K4-Pad3) -> /Pin_12
- K4 pad 4: unconnected-(K4-Pad4) -> /Pin_24
- K4 pad 5: unconnected-(K4-Pad5) -> /Pin_10
- K4 pad 6: unconnected-(K4-Pad6) -> /Pin_23
- K4 pad 7: unconnected-(K4-Pad7) -> /Pin_11
Routing:
- net (no net): track 0.00 -> 291.3 mm
- net /PT3 out: track 52.7 -> 0.00 mm
- net /PT4 out: track 48.3 -> 0.00 mm
- net /PT2 in: track 46.6 -> 0.00 mm, vias 1 -> 0
- net /PT3 in: track 41.0 -> 0.00 mm, vias 1 -> 0
- net /PT4 in: track 38.8 -> 0.00 mm
- net /PT1 out: track 25.6 -> 0.00 mm
- net /PT2 out: track 25.5 -> 0.00 mm
- net /PT1 in: track 12.7 -> 0.00 mm
- net /Pin_03: vias 0 -> 1
- net /Pin_02: vias 0 -> 1
