File: KiCAD/CIB - Sandbird Octopus.kicad_sch (KiCad schematic)
At the start: 51 parts, among them J1 DA15, J2 Molex, J3 PT 3-4, J4 PT 1-2, J5 Enable, J6 Pin Header, Q1 STN3NF06, Q2 STN3NF06, Q3 STN3NF06, Q4 STN3NF06, Q5 STN3NF06

Commit message: .
Parts:
- K1, K2, K3, K4, K5, K6, K7, K8: value ~ -> (none)
Other:
- note removed: "https://chargepoint.atlassian.net/wiki/spaces/EN/pages/5094740380/Pygmy+Octopus"

Commit message: .
Parts:
- removed J2: Molex, Connector_Molex:Molex_Micro-Fit_3.0_43045-1018_2x05-1MP_P3.00mm_Vertical, symbol Connector_Generic:Conn_02x05_Top_Bottom
- removed J3: PT 3-4, TerminalBlock_Phoenix:TerminalBlock_Phoenix_MPT-0,5-4-2.54_1x04_P2.54mm_Horizontal, symbol Connector:Screw_Terminal_01x04
- removed J4: PT 1-2, TerminalBlock_Phoenix:TerminalBlock_Phoenix_MPT-0,5-4-2.54_1x04_P2.54mm_Horizontal, symbol Connector:Screw_Terminal_01x04
- added D14, D15, D16: Red, LED_SMD:LED_0805_2012Metric_Pad1.15x1.40mm_HandSolder, symbol Device:LED_Small_Filled
- added Q6, Q7, Q8: STN3NF06, Package_TO_SOT_SMD:SOT-223-3_TabPin2, symbol Transistor_FET:NDT3055L
- added R19, R21, R22, R24, R25, R27: 1k, Resistor_SMD:R_0805_2012Metric_Pad1.20x1.40mm_HandSolder, symbol Device:R_Small
- added R20, R23, R26: 10k, Resistor_SMD:R_0805_2012Metric_Pad1.20x1.40mm_HandSolder, symbol Device:R_Small
- J1: value DA15 -> DB25; footprint Connector_Dsub:DSUB-9_Female_Horizontal_P2.77x2.84mm_EdgePinOffset7.70mm_Housed_MountingHolesOffset9.12mm -> Connector_Dsub:DSUB-25_Socket_Horizontal_P2.77x2.84mm_EdgePinOffset7.70mm_Housed_MountingHolesOffset9.12mm; symbol Connector:DE9_Receptacle_MountingHoles -> Connector:DB25_Socket_MountingHoles
- J6: value Pin Header -> Conn_01x26_Pin; footprint Connector_PinHeader_2.54mm:PinHeader_2x05_P2.54mm_Vertical -> Connector_PinHeader_2.54mm:PinHeader_2x013_P2.54mm_Vertical; symbol Connector:Conn_01x10_Pin -> Connector:Conn_01x26_Pin
Connections:
- net PT1 in is gone; now on net Pin_01: J1.1, J6.1 (Pin_1)
- net PT2 in is gone; now on net Pin_02: J1.2, J6.3 (Pin_3)
- net PT3 in is gone; now on net Pin_03: J1.3, J6.5 (Pin_5)
- net PT4 in is gone; now on net Pin_04: J1.4, J6.7 (Pin_7)
- net GND: now also J1.SH (PAD), J6.26 (Pin_26), D14.1 (K), D15.1 (K), D16.1 (K), Q6.3 (S), Q7.3 (S), Q8.3 (S), R20.2, R23.2, R26.2; no longer J1.0 (PAD), J6.10 (Pin_10)
- net Pin_05: now also K2.7
- net Relay_6: now also Q6.2 (D)
- net Relay_6_en: now also R19.1, R20.1, R21.1
- net Relay_7: now also Q7.2 (D)
- net Relay_7_en: now also R22.1, R23.1, R24.1
- net Relay_8: now also Q8.2 (D)
- net Relay_8_en: now also R25.1, R26.1, R27.1
- net Pin_16: now reaches K1.2
- net Pin_16: now also J1.16 (P16), J6.6 (Pin_6)
- net Pin_03: now reaches K1.3
- net Pin_15: now reaches K1.4
- net Pin_15: now also J1.15 (P15), J6.4 (Pin_4)
- net Pin_01: now reaches K1.5
- net Pin_14: now reaches K1.6
- net Pin_14: now also J1.14 (P14), J6.2 (Pin_2)
- net Pin_02: now reaches K1.7
- net Pin_25: now reaches K4.2
- net Pin_25: now also J1.25 (P25), J6.24 (Pin_24)
- net Pin_12: now reaches K4.3
- net Pin_12: now also J1.12, J6.23 (Pin_23)
- net Pin_24: now reaches K4.4
- net Pin_24: now also J1.24 (P24), J6.22 (Pin_22)
- net Pin_10: now reaches K4.5
- net Pin_10: now also J1.10, J6.19 (Pin_19)
- net Pin_23: now reaches K4.6
- net Pin_23: now also J1.23 (P23), J6.20 (Pin_20)
- net Pin_11: now reaches K4.7
- net Pin_11: now also J1.11, J6.21 (Pin_21)
- net Pin_19: now reaches K2.2
- net Pin_19: now also J1.19 (P19), J6.12 (Pin_12)
- net Pin_06: now reaches K2.3
- net Pin_06: now also J1.6, J6.11 (Pin_11)
- net Pin_18: now reaches K2.4
- net Pin_18: now also J1.18 (P18), J6.10 (Pin_10)
- net Pin_04: now reaches K2.5
- net Pin_17: now reaches K2.6
- net Pin_17: now also J1.17 (P17), J6.8 (Pin_8)
- net Pin_22: now reaches K3.2
- net Pin_22: now also J1.22 (P22), J6.18 (Pin_18)
- net Pin_09: now reaches K3.3
- net Pin_09: now also J1.9, J6.17 (Pin_17)
- net Pin_21: now reaches K3.4
- net Pin_21: now also J1.21 (P21), J6.16 (Pin_16)
- net Pin_07: now reaches K3.5
- net Pin_07: now also J1.7, J6.13 (Pin_13)
- net Pin_20: now reaches K3.6
- net Pin_20: now also J1.20 (P20), J6.14 (Pin_14)
- net Pin_08: now reaches K3.7
- net Pin_08: now also J1.8, J6.15 (Pin_15)
- removed net PT1 out: J1.6, J6.2 (Pin_2)
- removed net PT2 out: J1.7, J6.4 (Pin_4)
- removed net PT3 out: J1.8, J6.6 (Pin_6)
- removed net PT4 out: J1.9, J6.8 (Pin_8)
- new net: Q7.1 (G), R24.2
- new net: Q6.1 (G), R21.2
- new net: D15.2 (A), R22.2
- new net: D14.2 (A), R19.2
- new net: D16.2 (A), R25.2
- new net: Q8.1 (G), R27.2
- new net Pin_13: J1.13, J6.25 (Pin_25)
Other:
- note removed: "Swap this out for a D25"
- moved on the sheet: D10, D6, D7, D8, D9, J5, Q1, Q2, Q3, Q4, Q5, R10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
